Commit message: Fixing minor bugs

File: my_legged_robots_sims/urdf/monoped_controled.urdf (robot description, URDF)
Before this commit: robot monoped, 5 links, 4 joints
Links:
- link hipassembly: geometry collision mesh filename=package://my_legged_robots_description/meshes/leg/hipassemb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 scale=1 1 1; visual mesh filename=package://my_legged_robots_description/meshes/leg/hipassemb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 scale=1 1 1
- link lowerleg: geometry collision mesh filename=package://my_legged_robots_description/meshes/leg/lowerleg.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 scale=1 1 1; visual mesh filename=package://my_legged_robots_description/meshes/leg/lowerleg.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 scale=1 1 1
- link upperleg: geometry collision mesh filename=package://my_legged_robots_description/meshes/leg/upperleg.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 scale=1 1 1; visual mesh filename=package://my_legged_robots_description/meshes/leg/upperleg.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 scale=1 1 1
