Commit message: Added debug of some error spoted during AI testing

File: legged_robots_sims/urdf/monoped_controled.urdf (robot description, URDF)
Before this commit: robot monoped, 5 links, 4 joints
Links:
- link base: mass 0.4672 -> 31.5
- link contactsensor_link: mass 0.01 -> 0.8; geometry collision sphere radius=0.08; visual sphere radius=0.08
- link hipassembly: mass 0.1168 -> 7.5
- link lowerleg: mass 0.0292 -> 1.95
- link upperleg: mass 0.1168 -> 7.5
Joints:
- joint haa_joint: limit lower=-1.6 upper=1.6 effort=20 velocity=12.0 -> lower=-1.6 upper=1.6 effort=10000000 velocity=0.7
- joint hfe_joint: limit lower=-1.6 upper=1.6 effort=20 velocity=12.0 -> lower=-1.6 upper=1.6 effort=10000000 velocity=0.7
- joint kfe_joint: limit lower=-1.6 upper=0.0 effort=20 velocity=12.0 -> lower=-1.6 upper=0.0 effort=10000000 velocity=0.7
