Commit message: Added final controllers

File: legged_robots_sims/urdf/monoped_controled_2D.urdf (robot description, URDF)
Before this commit: robot monoped, 6 links, 5 joints
Joints:
- joint contactsensor_world_link_joint: axis (none) -> 0 0 1; limit (none) -> lower=-1.57 upper=1.57 effort=20 velocity=12.0; origin xyz=0 0 0.03 rpy=0.7 1.57 0 -> xyz=0 0 0.03 rpy=0.0 1.57 0; type fixed -> revolute
- joint haa_joint: limit lower=-1.6 upper=1.6 effort=20 velocity=12.0 -> lower=0.0 upper=0.0 effort=20 velocity=12.0
